Commit message: modified:   D1.urdf 	modified:   D1.urdf~ 	modified:   D2.urdf 	modified:   D2.urdf~ 	modified:   EXIT.urdf 	new file:   EXIT.urdf~ 	modified:   S1.urdf 	modified:   S1.urdf~ 	modified:   S2.urdf 	modified:   S2.urdf~

File: D1.urdf (robot description, URDF)
Before this commit: robot D1, 1 links, 0 joints
Links:
- link D1: geometry collision box size=0.5 0.5 0.0001; visual box size=0.5 0.5 0.0001

File: D2.urdf (robot description, URDF)
Before this commit: robot D2, 1 links, 0 joints
Links:
- link D2: geometry collision box size=0.1 0.1 0.0001; visual box size=0.1 0.1 0.0001

File: S1.urdf (robot description, URDF)
Before this commit: robot S1, 1 links, 0 joints
Links:
- link S1: geometry collision box size=0.5 0.5 0.0001; visual box size=0.5 0.5 0.0001

File: S2.urdf (robot description, URDF)
Before this commit: robot S2, 1 links, 0 joints
Links:
- link S2: geometry collision box size=0.5 0.5 0.0001; visual box size=0.5 0.5 0.0001

File: S3.urdf (robot description, URDF)
Before this commit: robot S3, 1 links, 0 joints
Links:
- link S3: geometry collision box size=0.5 0.5 0.0001; visual box size=0.5 0.5 0.0001
