Commit message: rearranged and modified files 	modified:   D2.urdf 	modified:   D2.urdf~ 	renamed:    brsu-c025-arena_original.urdf -> brsu-c025-arena.urdf 	modified:   brsu-c025-arena.urdf.xacro 	new file:   maze.urdf 	new file:   models/room.dae 	new file:   models/room.obj 	new file:   models/room.stl 	new file:   room.dae 	new file:   room.urdf 	renamed:    arena.launch -> trashed/arena.launch 	renamed:    arena.urdf -> trashed/arena.urdf

File: D2.urdf (robot description, URDF)
Before this commit: robot D2, 1 links, 0 joints
Links:
- link D2: geometry collision box size=0.5 0.5 0.0001; visual box size=0.5 0.5 0.0001

File: brsu-c025-arena.urdf.xacro (robot description, xacro)
@@ -12,26 +12,4 @@
 -->
 <robot name="brsu-c025-arena">
-	<link name="S1">
-    		<inertial>
-      			<origin xyz="1.042 0.766 0" />
-      			<mass value="10.0" />
-      			<inertia  ixx="1.0" ixy="0.0"  ixz="0.0"  iyy="1.0"  iyz="0.0"  izz="1.0" />
-    		</inertial>
-    		<visual>
-      			<origin xyz="1.042 0.766 0"/>
-      			<geometry>
-        			<box size="1 1 0.0001" />
-      			</geometry>
-			<material name="surface_pattern">
-				<texture filename="S1.jpg"/>
-			</material>
-    		</visual>
-    		<collision>
-      			<origin xyz="1.042 0.766 0"/>
-      		<geometry>
-        		<box size="1 1 0.0001" />
-      		</geometry>
-    		</collision>
-  	</link>
   	<link name="wall_1">
     		<inertial>

File: trashed/brsu-c025-arena.urdf.xacro (robot description, xacro)
@@ -12,4 +12,26 @@
 -->
 <robot name="brsu-c025-arena">
+	<link name="S1">
+    		<inertial>
+      			<origin xyz="1.042 0.766 0" />
+      			<mass value="10.0" />
+      			<inertia  ixx="1.0" ixy="0.0"  ixz="0.0"  iyy="1.0"  iyz="0.0"  izz="1.0" />
+    		</inertial>
+    		<visual>
+      			<origin xyz="1.042 0.766 0"/>
+      			<geometry>
+        			<box size="1 1 0.0001" />
+      			</geometry>
+			<material name="surface_pattern">
+				<texture filename="S1.jpg"/>
+			</material>
+    		</visual>
+    		<collision>
+      			<origin xyz="1.042 0.766 0"/>
+      		<geometry>
+        		<box size="1 1 0.0001" />
+      		</geometry>
+    		</collision>
+  	</link>
   	<link name="wall_1">
     		<inertial>
