Commit message: fiyed locations of D2, S2, fixed maze and room, all successfully spawned 	modified:   D2.urdf 	new file:   D2.urdf~ 	modified:   S2.urdf 	new file:   S2.urdf~ 	modified:   maze.urdf 	new file:   maze.urdf~ 	modified:   room.urdf 	new file:   room.urdf~

File: room.urdf (robot description, URDF)
Before this commit: robot room, 1 links, 0 joints
Links:
- link room: mass None -> 10.0; geometry collision mesh filename=/home/zinnirah/ros/workspace/edufill_component_zinnirah_wor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 scale=1 1 1; visual mesh filename=/home/zinnirah/ros/workspace/edufill_component_zinnirah_wor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 scale=1 1 1
