Commit message: urdfs to xacros, textures of D1, D2, S1, S2, S3, and EXIT are still not appearing. 	modified:   D1.urdf 	new file:   D1.urdf.xacro 	new file:   D2.urdf.xacro 	new file:   EXIT.urdf.xacro 	new file:   S1.urdf.xacro 	new file:   S2.urdf.xacro 	new file:   S3.urdf.xacro 	modified:   maze.urdf.xacro 	modified:   room.urdf.xacro

File: D2.urdf.xacro (robot description, xacro)
@@ -1,21 +1,21 @@
 <?xml version="1.0"?>
-<robot name="D1">
-	<link name="D1">
+<robot name="D2">
+	<link name="D2">
     		<inertial>
-      			<origin xyz="-0.99 -0.737 0" />
+      			<origin xyz="-0.99 0.737 0" />
       			<mass value="10.0" />
       			<inertia  ixx="1.0" ixy="0.0"  ixz="0.0"  iyy="1.0"  iyz="0.0"  izz="1.0" />
     		</inertial>
     		<visual>
-      			<origin xyz="-0.99 -0.737 0"/>
+      			<origin xyz="-0.99 0.737 0"/>
       			<geometry>
         			<box size="0.5 0.5 0.0001" />
       			</geometry>
 			<material name="surface">
-				<texture filename="D1.jpg" scale="0.01"/>
+				<texture filename="D2.jpg"/>
 			</material>
     		</visual>
     		<collision>
-      			<origin xyz="-0.99 -0.737 0"/>
+      			<origin xyz="-0.99 0.737 0"/>
       		<geometry>
         		<box size="0.5 0.5 0.0001" />

File: EXIT.urdf.xacro (robot description, xacro)
@@ -1,21 +1,21 @@
 <?xml version="1.0"?>
-<robot name="D1">
-	<link name="D1">
+<robot name="EXIT">
+	<link name="EXIT">
     		<inertial>
-      			<origin xyz="-0.99 -0.737 0" />
+      			<origin xyz="-2.165 0.05 0" />
       			<mass value="10.0" />
       			<inertia  ixx="1.0" ixy="0.0"  ixz="0.0"  iyy="1.0"  iyz="0.0"  izz="1.0" />
     		</inertial>
     		<visual>
-      			<origin xyz="-0.99 -0.737 0"/>
+      			<origin xyz="-2.165 0.05 0"/>
       			<geometry>
         			<box size="0.5 0.5 0.0001" />
       			</geometry>
 			<material name="surface">
-				<texture filename="D1.jpg" scale="0.01"/>
+				<texture filename="EXIT.jpg"/>
 			</material>
     		</visual>
     		<collision>
-      			<origin xyz="-0.99 -0.737 0"/>
+      			<origin xyz="-2.165 0.05 0"/>
       		<geometry>
         		<box size="0.5 0.5 0.0001" />

File: S1.urdf.xacro (robot description, xacro)
@@ -1,21 +1,21 @@
 <?xml version="1.0"?>
-<robot name="D1">
-	<link name="D1">
+<robot name="S1">
+	<link name="S1">
     		<inertial>
-      			<origin xyz="-0.99 -0.737 0" />
+      			<origin xyz="1.042 0.766 0" />
       			<mass value="10.0" />
       			<inertia  ixx="1.0" ixy="0.0"  ixz="0.0"  iyy="1.0"  iyz="0.0"  izz="1.0" />
     		</inertial>
     		<visual>
-      			<origin xyz="-0.99 -0.737 0"/>
+      			<origin xyz="1.042 0.766 0"/>
       			<geometry>
         			<box size="0.5 0.5 0.0001" />
       			</geometry>
 			<material name="surface">
-				<texture filename="D1.jpg" scale="0.01"/>
+				<texture filename="S1.jpg"/>
 			</material>
     		</visual>
     		<collision>
-      			<origin xyz="-0.99 -0.737 0"/>
+      			<origin xyz="1.042 0.766 0"/>
       		<geometry>
         		<box size="0.5 0.5 0.0001" />

File: S2.urdf.xacro (robot description, xacro)
@@ -1,21 +1,21 @@
 <?xml version="1.0"?>
-<robot name="D1">
-	<link name="D1">
+<robot name="S2">
+	<link name="S2">
     		<inertial>
-      			<origin xyz="-0.99 -0.737 0" />
+      			<origin xyz="1.041 -0.779 0" />
       			<mass value="10.0" />
       			<inertia  ixx="1.0" ixy="0.0"  ixz="0.0"  iyy="1.0"  iyz="0.0"  izz="1.0" />
     		</inertial>
     		<visual>
-      			<origin xyz="-0.99 -0.737 0"/>
+      			<origin xyz="1.041 -0.779 0"/>
       			<geometry>
         			<box size="0.5 0.5 0.0001" />
       			</geometry>
 			<material name="surface">
-				<texture filename="D1.jpg" scale="0.01"/>
+				<texture filename="S2.jpg"/>
 			</material>
     		</visual>
     		<collision>
-      			<origin xyz="-0.99 -0.737 0"/>
+      			<origin xyz="1.041 -0.779 0"/>
       		<geometry>
         		<box size="0.5 0.5 0.0001" />

File: S3.urdf.xacro (robot description, xacro)
@@ -1,21 +1,21 @@
 <?xml version="1.0"?>
-<robot name="D1">
-	<link name="D1">
+<robot name="S3">
+	<link name="S3">
     		<inertial>
-      			<origin xyz="-0.99 -0.737 0" />
+      			<origin xyz="1.082 0.01 0" />
       			<mass value="10.0" />
       			<inertia  ixx="1.0" ixy="0.0"  ixz="0.0"  iyy="1.0"  iyz="0.0"  izz="1.0" />
     		</inertial>
     		<visual>
-      			<origin xyz="-0.99 -0.737 0"/>
+      			<origin xyz="1.082 0.01 0"/>
       			<geometry>
         			<box size="0.5 0.5 0.0001" />
       			</geometry>
 			<material name="surface">
-				<texture filename="D1.jpg" scale="0.01"/>
+				<texture filename="S3.jpg"/>
 			</material>
     		</visual>
     		<collision>
-      			<origin xyz="-0.99 -0.737 0"/>
+      			<origin xyz="1.082 0.01 0"/>
       		<geometry>
         		<box size="0.5 0.5 0.0001" />

File: maze.urdf.xacro (robot description, xacro)
@@ -1,10 +1,21 @@
 <?xml version="1.0"?>
-<robot name="maze">
+<robot name="maze" static="true">
 	<link name="maze">
+		<inertial>
+			<origin xyz="0 0 1"/>
+			<mass value="10.0"/>
+			<inertia ixx="1.0" ixy="0.0" ixz="0.0" iyy="1.0" iyz="0.0" izz="1.0"/>
+		</inertial>
+		<collision name="room_collision">
+            		<geometry>
+                		<mesh filename="/home/zinnirah/ros/workspace/edufill_component_zinnirah_workspace/maze_wide.dae" scale="1 1 1"/>
+            		</geometry>
+        	</collision>
 		<visual>
 			<geometry>
-				<mesh filename= "maze_wide.dae"/>
+				<mesh filename= "/home/zinnirah/ros/workspace/edufill_component_zinnirah_workspace/maze_wide.dae" scale="1 1 1"/>
 			</geometry>
 		</visual>
 	</link>
+	</link>
 </robot>
