Commit message: fixed issues, untested

File: D1.urdf.xacro (robot description, xacro)
@@ -1,22 +1,22 @@
 <?xml version="1.0"?>
-<robot name="edufill_EXIT">
-<xacro:macro name="edufill_EXIT" params="name">
-	<link name="edufill_EXIT">
+<robot name="edufill_D1">
+<xacro:macro name="edufill_D1" params="name">
+	<link name="edufill_D1">
     		<inertial>
-      			<origin xyz="-2.165 0.05 0" />
+      			<origin xyz="-0.99 -0.737 0" />
       			<mass value="10.0" />
       			<inertia  ixx="1.0" ixy="0.0"  ixz="0.0"  iyy="1.0"  iyz="0.0"  izz="1.0" />
     		</inertial>
     		<visual>
-      			<origin xyz="-2.165 0.05 0"/>
+      			<origin xyz="-0.99 -0.737 0"/>
       			<geometry>
         			<box size="0.5 0.5 0.0001" />
       			</geometry>
 			<material name="surface">
-				<texture filename="package://edufill_gazebo_world/common/worlds/EXIT.jpg"/>
+				<texture filename="package://edufill_gazebo_world/common/worlds/D1.jpg" scale="0.01"/>
 			</material>
     		</visual>
     		<collision>
-      			<origin xyz="-2.165 0.05 0"/>
+      			<origin xyz="-0.99 -0.737 0"/>
       		<geometry>
         		<box size="0.5 0.5 0.0001" />
@@ -25,4 +25,4 @@
   	</link>
 </xacro:macro>
-<xacro:edufill_EXIT name="edufill_EXIT" />
+<xacro:edufill_D1 name="edufill_D1" />
 </robot>

File: D2.urdf.xacro (robot description, xacro)
@@ -1,5 +1,6 @@
 <?xml version="1.0"?>
-<robot name="D2">
-	<link name="D2">
+<robot name="edufill_D2">
+<xacro:macro name="edufill_D2" params="name">
+	<link name="edufill_D2">
     		<inertial>
       			<origin xyz="-0.99 0.737 0" />
@@ -13,5 +14,5 @@
       			</geometry>
 			<material name="surface">
-				<texture filename="D2.jpg"/>
+				<texture filename="package://edufill_gazebo_world/common/worlds/D2.jpg"/>
 			</material>
     		</visual>
@@ -23,3 +24,5 @@
     		</collision>
   	</link>
+</xacro:macro>
+<xacro:edufill_D2 name="edufill_D2" />
 </robot>

File: S1.urdf.xacro (robot description, xacro)
@@ -1,5 +1,6 @@
 <?xml version="1.0"?>
-<robot name="S1">
-	<link name="S1">
+<robot name="edufill_S1">
+<xacro:macro name="edufill_S1" params="name">
+	<link name="edufill_S1">
     		<inertial>
       			<origin xyz="1.042 0.766 0" />
@@ -13,5 +14,5 @@
       			</geometry>
 			<material name="surface">
-				<texture filename="S1.jpg"/>
+				<texture filename="package://edufill_gazebo_world/common/worlds/S1.jpg"/>
 			</material>
     		</visual>
@@ -23,3 +24,5 @@
     		</collision>
   	</link>
+</xacro:macro>
+<xacro:edufill_S1 name="edufill_S1" />
 </robot>

File: S2.urdf.xacro (robot description, xacro)
@@ -1,5 +1,6 @@
 <?xml version="1.0"?>
-<robot name="S2">
-	<link name="S2">
+<robot name="edufill_S2">
+<xacro:macro name="edufill_S2" params="name">
+	<link name="edufill_S2">
     		<inertial>
       			<origin xyz="1.041 -0.779 0" />
@@ -13,5 +14,5 @@
       			</geometry>
 			<material name="surface">
-				<texture filename="S2.jpg"/>
+				<texture filename="package://edufill_gazebo_world/common/worlds/S2.jpg"/>
 			</material>
     		</visual>
@@ -23,3 +24,5 @@
     		</collision>
   	</link>
+</xacro:macro>
+<xacro:edufill_S2 name="edufill_S2" />
 </robot>

File: S3.urdf.xacro (robot description, xacro)
@@ -1,5 +1,6 @@
 <?xml version="1.0"?>
-<robot name="S3">
-	<link name="S3">
+<robot name="edufill_S3">
+<xacro:macro name="edufill_S3" params="name">
+	<link name="edufill_S3">
     		<inertial>
       			<origin xyz="1.082 0.01 0" />
@@ -13,5 +14,5 @@
       			</geometry>
 			<material name="surface">
-				<texture filename="S3.jpg"/>
+				<texture filename="package://edufill_gazebo_world/common/worlds/S3.jpg"/>
 			</material>
     		</visual>
@@ -23,3 +24,5 @@
     		</collision>
   	</link>
+</xacro:macro>
+<xacro:edufill_S3 name="edufill_S3" />
 </robot>

File: maze.urdf.xacro (robot description, xacro)
@@ -8,12 +8,12 @@
 			<inertia ixx="1.0" ixy="0.0" ixz="0.0" iyy="1.0" iyz="0.0" izz="1.0"/>
 		</inertial>
-		<collision name="room_collision">
+		<collision name="maze_collision">
             		<geometry>
-                		<mesh filename="package://$(find edufill_gazebo_world)/common/worlds/edufill_maze.dae" scale="1 1 1"/>
+                		<mesh filename="package://edufill_gazebo_world/common/worlds/edufill_maze.dae" scale="1 1 1"/>
             		</geometry>
         	</collision>
 		<visual>
 			<geometry>
-				<mesh filename= "package://$(find edufill_gazebo_world)/common/worlds/edufill_maze.dae" scale="1 1 1"/>
+				<mesh filename= "package://edufill_gazebo_world/common/worlds/edufill_maze.dae" scale="1 1 1"/>
 			</geometry>
 		</visual>
